File: hardware/beeper.kicad_pcb (KiCad board)
At the start: 2 copper layers, 50.3 x 50.3 mm, 20 parts, among them J1 AVR-ISP-6, SW1 SW_Push, U1 ATtiny861A-PU, U2 SN76489

Commit message: shorter traces
Parts:
- C2: footprint Capacitor_THT:CP_Radial_D8.0mm_P5.00mm -> Capacitor_THT:CP_Radial_D6.3mm_P2.50mm
- moved C2 1.98 mm to (176.7, 121.8)
Routing:
- net Net-(U1-Pad8): track 47.7 -> 16.1 mm
- net Net-(U1-Pad7): track 48.4 -> 23.7 mm
- net Net-(J1-Pad1): track 43.1 -> 25.6 mm
- net VCC: track 76.5 -> 64.6 mm
- net Net-(U1-Pad12): track 25.3 -> 15.8 mm
- net Net-(J1-Pad5): track 42.8 -> 34.1 mm
- net Net-(U1-Pad11): track 29.3 -> 23.3 mm
- net Net-(SW1-Pad1): track 47.5 -> 42.4 mm
- net Net-(C2-Pad1): track 29.1 -> 25.6 mm
- net Net-(J1-Pad4): track 21.1 -> 19.4 mm
- net Net-(C2-Pad2): track 6.43 -> 8.11 mm
- net Net-(LED4-Pad2): track 24.2 -> 23.1 mm
- net Net-(U1-Pad13): track 19.3 -> 20.2 mm
- net Net-(J1-Pad3): track 34.7 -> 33.9 mm
Other:
- board text added: "music_box v0.2 by Jeremy Stanley 2021-02"
- board text removed: "music_box v0.1 by @jstanley0 2021-02"
