File: hardware/beeper.sch (KiCad schematic (older format))
At the start: 16 parts, among them J1 AVR-ISP-6, SW1 SW_Push, U1 ATtiny861A-PU, U2 SN76489

Commit message: shorter traces
Parts:
- C2: footprint Capacitor_THT:CP_Radial_D8.0mm_P5.00mm -> Capacitor_THT:CP_Radial_D6.3mm_P2.50mm
Changed lines of the file:
@@
 F 0 "C2" H 7715 3546 50  0000 L CNN
 F 1 "10uF" H 7715 3455 50  0000 L CNN
-F 2 "Capacitor_THT:CP_Radial_D8.0mm_P5.00mm" H 7600 3500 50  0001 C CNN
+F 2 "Capacitor_THT:CP_Radial_D6.3mm_P2.50mm" H 7600 3500 50  0001 C CNN
 F 3 "~" H 7600 3500 50  0001 C CNN
 	1    7600 3500
